File: smartmeter-ir-reader.kicad_pcb (KiCad board)
At the start: 2 copper layers, 2 parts

Commit message: Initial version
Parts:
- removed the G*** at (22.4, 182.3)
- added C1: 1uF, Capacitor_SMD:C_0603_1608Metric_Pad1.08x0.95mm_HandSolder, F.Cu at (139.0, 99.9)
- added C2: 1uF, Capacitor_SMD:C_0603_1608Metric_Pad1.08x0.95mm_HandSolder, F.Cu at (151.7, 105.5)
- added C3: 1uF, Capacitor_SMD:C_0603_1608Metric_Pad1.08x0.95mm_HandSolder, F.Cu at (158.2, 99.3)
- added D1: BAT46W, Diode_SMD:D_SOD-123, F.Cu at (157.5, 109.7)
- added D2: LED, LED_THT:LED_D3.0mm_Clear, B.Cu at (146.8, 103.1)
- added IC1: SN74LVC1G17DBVR, Chof747 Footprints:SOT95P270X145-5N, F.Cu at (158.2, 102.4)
- added IC2: SN74LVC1G17DBVR, Chof747 Footprints:SOT95P270X145-5N, F.Cu at (139.0, 103.1)
- added J1: RJ10, Connector_RJ:RJ12_Amphenol_54601, F.Cu at (145.7, 111.7)
- added Q1: S8050, Package_TO_SOT_SMD:SOT-23, F.Cu at (152.4, 98.4)
- added Q2: S8550, Package_TO_SOT_SMD:SOT-23, F.Cu at (145.5, 98.8)
- added Q3: SFH309, LED_THT:LED_D3.0mm_Clear, B.Cu at (150.8, 103.1)
- added R1: 10k, Resistor_SMD:R_0603_1608Metric_Pad0.98x0.95mm_HandSolder, F.Cu at (152.5, 94.6)
- added R2: 10k, Resistor_SMD:R_0603_1608Metric_Pad0.98x0.95mm_HandSolder, F.Cu at (154.2, 94.6)
- added R3: 10k, Resistor_SMD:R_0603_1608Metric_Pad0.98x0.95mm_HandSolder, F.Cu at (147.3, 95.3)
- added R4: 180, Resistor_SMD:R_0603_1608Metric_Pad0.98x0.95mm_HandSolder, F.Cu at (146.9, 106.7)
- moved G*** 135.5 mm to (139.2, 104.1)
Routing:
- net +3V3: track 0.00 -> 61.3 mm
- net /RX: track 0.00 -> 27.4 mm
- net Net-(IC1-A): track 0.00 -> 15.8 mm
- net Net-(IC2-Y): track 0.00 -> 13.4 mm
- net /TX: track 0.00 -> 12.8 mm
- net /VCC: track 0.00 -> 11.8 mm
- net GND: track 0.00 -> 9.49 mm, vias 0 -> 8
- net Net-(Q1-B): track 0.00 -> 7.88 mm
- net Net-(D2-A): track 0.00 -> 4.41 mm
- net Net-(D2-K): track 0.00 -> 2.73 mm
- net Net-(Q2-B): track 0.00 -> 2.51 mm
- added copper zone on B.Cu, net GND
Other:
- board outline added: 27 x 34.8 mm
- board text added: "Smart-Meter-IR"
- board text added: "v1.0 (2023)"

Commit message: Initial version Revision 1.0
Routing:
- added copper zone on B.Cu, net +3V3
Other:
- outline, holes or cut-outs redrawn
Changed lines of the file:
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@@
       (stroke (width 0) (type solid)) (fill solid) (layer "B.SilkS"))
   )
+  (gr_line (start 150.8436 104.8932) (end 150.8436 101.2932)
+    (stroke (width 0.15) (type default)) (layer "Dwgs.User"))
   (gr_poly
     (pts
@@
       (xy 140.104285 113.362388)
       (xy 140.674148 113.820456)
-      (xy 141.267975 114.247001)
-      (xy 141.644 114.5232)
-      (xy 141.634 124.3432)
-      (xy 156.054 124.3432)
-      (xy 156.054 114.5132)
-      (xy 156.420025 114.247001)
+      (xy 141.054 114.1732)
+      (xy 141.054 124.3332)
+      (xy 156.544 124.2632)
+      (xy 156.544 114.247001)
       (xy 157.013852 113.820456)
       (xy 157.583715 113.362388)
@@
     (effects (font (size 1.5 1.5) (thickness 0.3) bold) (justify left bottom mirror))
   )
-  (gr_text "Smart-Meter-IR" (at 183.874 86.2357) (layer "B.SilkS")
+  (gr_text "Smart-Meter-IR" (at 157.874 97.0732) (layer "B.SilkS")
     (effects (font (size 1.5 1.5) (thickness 0.3) bold) (justify left bottom mirror))
   )
@@
   (segment (start 147.4836 99.7132) (end 146.4215 99.7132) (width 0.25) (layer "F.Cu") (net 1))
   (segment (start 154.244 93.7207) (end 155.3465 93.7207) (width 0.25) (layer "F.Cu") (net 2))
+  (segment (start 140.334 104.3332) (end 139.934 104.3332) (width 0.25) (layer "F.Cu") (net 2))
+  (segment (start 140.964 104.9632) (end 140.334 104.3332) (width 0.25) (layer "F.Cu") (net 2))
   (segment (start 151.494 99.3732) (end 150.814 99.3732) (width 0.25) (layer "F.Cu") (net 2))
   (segment (start 159.124 98.0732) (end 159.124 99.2757) (width 0.25) (layer "F.Cu") (net 2))
   (segment (start 150.814 99.3732) (end 150.494 99.6932) (width 0.25) (layer "F.Cu") (net 2))
-  (segment (start 140.854 104.3332) (end 140.904 104.3832) (width 0.25) (layer "F.Cu") (net 2))
   (segment (start 159.124 99.2757) (end 159.1065 99.2932) (width 0.25) (layer "F.Cu") (net 2))
   (segment (start 139.864 98.7332) (end 139.864 99.8857) (width 0.25) (layer "F.Cu") (net 2))
-  (segment (start 139.934 104.3332) (end 140.854 104.3332) (width 0.25) (layer "F.Cu") (net 2))
   (segment (start 145.834 107.6032) (end 146.9165 107.6032) (width 0.25) (layer "F.Cu") (net 2))
   (segment (start 159.174 103.6832) (end 159.174 105.0832) (width 0.25) (layer "F.Cu") (net 2))
@@
   (via (at 159.164 105.0932) (size 0.8) (drill 0.4) (layers "F.Cu" "B.Cu") (free) (net 2))
   (via (at 145.834 107.6032) (size 0.8) (drill 0.4) (layers "F.Cu" "B.Cu") (free) (net 2))
-  (via (at 140.904 104.3832) (size 0.8) (drill 0.4) (layers "F.Cu" "B.Cu") (free) (net 2))
+  (via (at 140.964 104.9632) (size 0.8) (drill 0.4) (layers "F.Cu" "B.Cu") (free) (net 2))
   (via (at 159.124 98.0732) (size 0.8) (drill 0.4) (layers "F.Cu" "B.Cu") (free) (net 2))
   (via (at 150.494 99.6932) (size 0.8) (drill 0.4) (layers "F.Cu" "B.Cu") (net 2))
@@
   (segment (start 145.074 94.4432) (end 141.294 98.2232) (width 0.13) (layer "F.Cu") (net 11))
   (segment (start 141.294 101.1332) (end 140.594 101.8332) (width 0.13) (layer "F.Cu") (net 11))
+  (zone (net 1) (net_name "+3V3") (layer "B.Cu") (hatch edge 0.5)
+    (priority 1)
+    (connect_pads yes (clearance 0.508))
+    (min_thickness 0.25) (filled_areas_thickness no)
+    (fill yes (thermal_gap 0.5) (thermal_bridge_width 0.5))
+    (polygon
+      (pts
+        (xy 151.744 100.8332)
+        (xy 148.254 100.8132)
+        (xy 148.264 104.8732)
+        (xy 151.744 104.8732)
+      )
+    )
+  )
   (zone (net 2) (net_name "GND") (layer "B.Cu") (hatch edge 0.5)
     (connect_pads (clearance 0.508))

Commit message: corrected RJ12 socket Connector
Connections:
- J1 pad 1: GND -> (no net)
- J1 pad 5: (no net) -> GND
Other:
- board text added: "v1.1 (2023)"
- board text removed: "v1.0 (2023)"
Changed lines of the file:
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@@
     (property "Sheetfile" "smartmeter-ir-reader.kicad_sch")
     (property "Sheetname" "")
-    (property "ki_description" "RJ connector, 4P4C (4 positions 4 connected)")
+    (property "ki_description" "RJ connector, 4P4C (4 positions 4 connected), RJ9/RJ10/RJ22")
     (property "ki_keywords" "4P4C RJ socket connector")
     (attr through_hole)
@@
     (pad "" np_thru_hole circle locked (at -1.91 8.89) (size 3.25 3.25) (drill 3.25) (layers "*.Cu" "*.Mask"))
     (pad "" np_thru_hole circle locked (at 8.25 8.89) (size 3.25 3.25) (drill 3.25) (layers "*.Cu" "*.Mask"))
-    (pad "1" thru_hole rect locked (at 0 0) (size 1.52 1.52) (drill 0.76) (layers "*.Cu" "*.Mask")
-      (net 2 "GND") (pintype "passive"))
+    (pad "1" thru_hole rect locked (at 0 0) (size 1.52 1.52) (drill 0.76) (layers "*.Cu" "*.Mask"))
     (pad "2" thru_hole circle locked (at 1.27 2.54) (size 1.52 1.52) (drill 0.76) (layers "*.Cu" "*.Mask")
       (net 6 "/RX") (pintype "passive"))
@@
     (pad "4" thru_hole circle locked (at 3.81 2.54) (size 1.52 1.52) (drill 0.76) (layers "*.Cu" "*.Mask")
       (net 3 "/VCC") (pintype "passive"))
-    (pad "5" thru_hole circle locked (at 5.08 0) (size 1.52 1.52) (drill 0.76) (layers "*.Cu" "*.Mask"))
+    (pad "5" thru_hole circle locked (at 5.08 0) (size 1.52 1.52) (drill 0.76) (layers "*.Cu" "*.Mask")
+      (net 2 "GND") (pintype "passive"))
     (pad "6" thru_hole circle locked (at 6.35 2.54) (size 1.52 1.52) (drill 0.76) (layers "*.Cu" "*.Mask"))
     (model ":USERMODELS:3dmodels/RJ12-Connector.step"
@@
     )
     (stroke (width 0.2) (type solid)) (fill none) (layer "Edge.Cuts"))
-  (gr_text "v1.0 (2023)" (at 155.544 117.9332) (layer "B.SilkS")
+  (gr_text "v1.1 (2023)" (at 155.544 117.9332) (layer "B.SilkS")
     (effects (font (size 1.5 1.5) (thickness 0.3) bold) (justify left bottom mirror))
   )

Commit message: V1.2 with corrected transistor layouts
Parts:
- Q1: value S8050 -> SS8050-G
- moved R3 2.00 mm to (145.4, 94.6), turned to -90 degrees
- moved Q2 0.33 mm to (145.5, 98.4), turned to 0 degrees
- turned Q1 to 0 degrees
Connections:
- Q1 pad 1: GND -> Net-(Q1-B)
- Q1 pad 2: Net-(Q1-B) -> GND
- Q2 pad 1: +3V3 -> Net-(Q2-B)
- Q2 pad 2: Net-(Q2-B) -> +3V3
Routing:
- net Net-(Q1-B): track 7.88 -> 13.5 mm
- net Net-(D2-A): track 4.41 -> 8.62 mm
- net +3V3: track 61.3 -> 63.1 mm
- net Net-(IC1-A): track 15.8 -> 17.6 mm
- net Net-(IC2-Y): track 13.4 -> 12.3 mm
- net GND: track 9.79 -> 10.4 mm
Other:
- board size 27 x 34.8 mm -> 27 x 34.7 mm
- board text added: "G"
- board text added: "RX"
- board text added: "TX"
- board text added: "V+"
- board text added: "v1.2 (2023)"
- board text removed: "v1.1 (2023)"
